File: board files/strain gauges/BETA/minimal/minimal.kicad_pcb (KiCad board)
At the start: 2 copper layers, 24 x 36.7 mm, 10 parts, among them J1 PR&J

Commit message: fixed strain gauge routing, added images of all boards
Routing:
- net GND: track 0.00 -> 97.8 mm
- removed copper zone on B.Cu, net GND
- removed copper zone on F.Cu, net GND
Changed lines of the file:
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@@
     (fp_arc (start 6.658126 4.625) (mid 6.674001 4.703822) (end 6.686135 4.783306)
       (stroke (width 0.2) (type solid)) (layer "Cmts.User"))
-    (fp_arc (start 6.686135 -4.783307) (mid 6.674002 -4.703822) (end 6.658126 -4.625)
+    (fp_arc (start 6.686135 -4.783307) (mid 6.674003 -4.703822) (end 6.658126 -4.625)
       (stroke (width 0.2) (type solid)) (layer "Cmts.User"))
     (fp_arc (start 6.686135 4.783306) (mid 6.61145 6.611448) (end 4.783308 6.686133)
@@
   (gr_rect (start 0 0) (end 24 36.7)
     (stroke (width 0.2) (type default)) (fill none) (layer "Edge.Cuts"))
+  (segment (start 12 3.1) (end 11.6 3.5) (width 0.25) (layer "F.Cu") (net 1))
+  (segment (start 6.343146 21.856854) (end 6.343146 19.806854) (width 0.25) (layer "F.Cu") (net 1))
+  (segment (start 8.736292 22.2) (end 6.343146 19.806854) (width 0.25) (layer "F.Cu") (net 1))
+  (segment (start 20.631891 3.5) (end 20.631891 24.768109) (width 0.25) (layer "F.Cu") (net 1))
+  (segment (start 12 22.2) (end 8.736292 22.2) (width 0.25) (layer "F.Cu") (net 1))
+  (segment (start 20.631891 3.5) (end 17.656854 6.475037) (width 0.25) (layer "F.Cu") (net 1))
+  (segment (start 12 14.15) (end 7.75 9.9) (width 0.25) (layer "F.Cu") (net 1))
+  (segment (start 8.26 29.66) (end 8.26 34.3) (width 0.25) (layer "F.Cu") (net 1))
+  (segment (start 3.431891 3.5) (end 7 7.068109) (width 0.25) (layer "F.Cu") (net 1))
+  (segment (start 3.4 24.8) (end 6.343146 21.856854) (width 0.25) (layer "F.Cu") (net 1))
+  (segment (start 17.656854 6.475037) (end 17.656854 8.493146) (width 0.25) (layer "F.Cu") (net 1))
+  (segment (start 7 18.4) (end 11.25 14.15) (width 0.25) (layer "F.Cu") (net 1))
+  (segment (start 17 18.4) (end 12.75 14.15) (width 0.25) (layer "F.Cu") (net 1))
+  (segment (start 12.4 3.5) (end 12 3.1) (width 0.25) (layer "F.Cu") (net 1))
+  (segment (start 20.631891 24.768109) (end 20.6 24.8) (width 0.25) (layer "F.Cu") (net 1))
+  (segment (start 12.75 14.15) (end 12 14.15) (width 0.25) (layer "F.Cu") (net 1))
+  (segment (start 11.25 14.15) (end 12 14.15) (width 0.25) (layer "F.Cu") (net 1))
+  (segment (start 3.4 24.8) (end 8.26 29.66) (width 0.25) (layer "F.Cu") (net 1))
+  (segment (start 18.606891 3.5) (end 12.4 3.5) (width 0.25) (layer "F.Cu") (net 1))
+  (segment (start 7 7.068109) (end 7 9.15) (width 0.25) (layer "F.Cu") (net 1))
+  (segment (start 7.75 9.9) (end 7 9.9) (width 0.25) (layer "F.Cu") (net 1))
+  (segment (start 11.6 3.5) (end 3.431891 3.5) (width 0.25) (layer "F.Cu") (net 1))
   (via (at 12 22.2) (size 0.8) (drill 0.4) (layers "F.Cu" "B.Cu") (free) (net 1))
+  (segment (start 12 22.2) (end 12 25.2) (width 0.25) (layer "B.Cu") (net 1))
   (segment (start 12 24.55) (end 12 33.1) (width 0.25) (layer "F.Cu") (net 2))
   (segment (start 12 33.1) (end 10.8 34.3) (width 0.25) (layer "F.Cu") (net 2))
@@
   (segment (start 19.806854 16.769354) (end 19.806854 20.697414) (width 0.2) (layer "B.Cu") (net 4))
   (segment (start 12 8.9625) (end 19.806854 16.769354) (width 0.2) (layer "B.Cu") (net 4))
-  (zone (net 1) (net_name "GND") (layers "F&B.Cu") (hatch edge 0.5)
-    (connect_pads (clearance 0.5))
-    (min_thickness 0.25) (filled_areas_thickness no)
-    (fill yes (thermal_gap 0.5) (thermal_bridge_width 0.5))
-    (polygon
-      (pts
-        (xy 24 -0.1)
-        (xy 0 -0.1)
-        (xy 0 36.7)
-        (xy 24 36.7)
-      )
-    )
-  )
 )
