File: hardware/board files/strain gauges/BETA/minimal/minimal.kicad_pcb (KiCad board)
At the start: 2 copper layers, 24 x 36.8 mm, 10 parts, among them J1 PR&J

Commit message: finalized boards for production
Changed lines of the file:
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@@
   )
   (setup
+    (stackup
+      (layer "F.SilkS" (type "Top Silk Screen"))
+      (layer "F.Paste" (type "Top Solder Paste"))
+      (layer "F.Mask" (type "Top Solder Mask") (thickness 0.01))
+      (layer "F.Cu" (type "copper") (thickness 0.035))
+      (layer "dielectric 1" (type "core") (thickness 1.51) (material "FR4") (epsilon_r 4.5) (loss_tangent 0.02))
+      (layer "B.Cu" (type "copper") (thickness 0.035))
+      (layer "B.Mask" (type "Bottom Solder Mask") (thickness 0.01))
+      (layer "B.Paste" (type "Bottom Solder Paste"))
+      (layer "B.SilkS" (type "Bottom Silk Screen"))
+      (copper_finish "None")
+      (dielectric_constraints no)
+    )
     (pad_to_mask_clearance 0)
     (pcbplotparams
@@
     (fp_line (start 3.15 1.6) (end -3.15 1.6)
       (stroke (width 0.1) (type solid)) (layer "F.Fab"))
-    (pad "1" smd roundrect (at -2.9625 0 90) (size 1.225 3.35) (layers "F.Cu" "F.Paste" "F.Mask") (roundrect_rratio 0.204082)
+    (pad "1" smd roundrect (at -2.9625 0 90) (size 1.225 3.35) (layers "F.Cu" "F.Paste" "F.Mask") (roundrect_rratio 0.2040816327)
       (net 4 "IN-") (pintype "passive"))
-    (pad "2" smd roundrect (at 2.9625 0 90) (size 1.225 3.35) (layers "F.Cu" "F.Paste" "F.Mask") (roundrect_rratio 0.204082)
+    (pad "2" smd roundrect (at 2.9625 0 90) (size 1.225 3.35) (layers "F.Cu" "F.Paste" "F.Mask") (roundrect_rratio 0.2040816327)
       (net 1 "GND") (pintype "passive"))
     (model "${KICAD6_3DMODEL_DIR}/Resistor_SMD.3dshapes/R_2512_6332Metric.wrl"
@@
     (fp_arc (start 6.658126 4.625) (mid 6.674001 4.703822) (end 6.686135 4.783306)
       (stroke (width 0.2) (type solid)) (layer "Cmts.User"))
-    (fp_arc (start 6.686135 -4.783307) (mid 6.674003 -4.703822) (end 6.658126 -4.625)
+    (fp_arc (start 6.686135 -4.783307) (mid 6.674002 -4.703822) (end 6.658126 -4.625)
       (stroke (width 0.2) (type solid)) (layer "Cmts.User"))
     (fp_arc (start 6.686135 4.783306) (mid 6.61145 6.611448) (end 4.783308 6.686133)
@@
     (fp_line (start 3.15 1.6) (end -3.15 1.6)
       (stroke (width 0.1) (type solid)) (layer "F.Fab"))
-    (pad "1" smd roundrect (at -2.9625 0 90) (size 1.225 3.35) (layers "F.Cu" "F.Paste" "F.Mask") (roundrect_rratio 0.204082)
+    (pad "1" smd roundrect (at -2.9625 0 90) (size 1.225 3.35) (layers "F.Cu" "F.Paste" "F.Mask") (roundrect_rratio 0.2040816327)
       (net 2 "VDDA") (pintype "passive"))
-    (pad "2" smd roundrect (at 2.9625 0 90) (size 1.225 3.35) (layers "F.Cu" "F.Paste" "F.Mask") (roundrect_rratio 0.204082)
+    (pad "2" smd roundrect (at 2.9625 0 90) (size 1.225 3.35) (layers "F.Cu" "F.Paste" "F.Mask") (roundrect_rratio 0.2040816327)
       (net 3 "IN+") (pintype "passive"))
     (model "${KICAD6_3DMODEL_DIR}/Resistor_SMD.3dshapes/R_2512_6332Metric.wrl"
@@
     (fp_line (start 3.15 1.6) (end 3.15 -1.6)
       (stroke (width 0.1) (type solid)) (layer "B.Fab"))
-    (pad "1" smd roundrect (at -2.9625 0 90) (size 1.225 3.35) (layers "B.Cu" "B.Paste" "B.Mask") (roundrect_rratio 0.204082)
+    (pad "1" smd roundrect (at -2.9625 0 90) (size 1.225 3.35) (layers "B.Cu" "B.Paste" "B.Mask") (roundrect_rratio 0.2040816327)
       (net 1 "GND") (pintype "passive"))
-    (pad "2" smd roundrect (at 2.9625 0 90) (size 1.225 3.35) (layers "B.Cu" "B.Paste" "B.Mask") (roundrect_rratio 0.204082)
+    (pad "2" smd roundrect (at 2.9625 0 90) (size 1.225 3.35) (layers "B.Cu" "B.Paste" "B.Mask") (roundrect_rratio 0.2040816327)
       (net 3 "IN+") (pintype "passive"))
     (model "${KICAD6_3DMODEL_DIR}/Resistor_SMD.3dshapes/R_2512_6332Metric.wrl"
@@
     (fp_line (start 3.15 1.6) (end 3.15 -1.6)
       (stroke (width 0.1) (type solid)) (layer "B.Fab"))
-    (pad "1" smd roundrect (at -2.9625 0 90) (size 1.225 3.35) (layers "B.Cu" "B.Paste" "B.Mask") (roundrect_rratio 0.204082)
+    (pad "1" smd roundrect (at -2.9625 0 90) (size 1.225 3.35) (layers "B.Cu" "B.Paste" "B.Mask") (roundrect_rratio 0.2040816327)
       (net 4 "IN-") (pintype "passive"))
-    (pad "2" smd roundrect (at 2.9625 0 90) (size 1.225 3.35) (layers "B.Cu" "B.Paste" "B.Mask") (roundrect_rratio 0.204082)
+    (pad "2" smd roundrect (at 2.9625 0 90) (size 1.225 3.35) (layers "B.Cu" "B.Paste" "B.Mask") (roundrect_rratio 0.2040816327)
       (net 2 "VDDA") (pintype "passive"))
     (model "${KICAD6_3DMODEL_DIR}/Resistor_SMD.3dshapes/R_2512_6332Metric.wrl"

Commit message: added cad and stl files for initial test version of a modified stealthburner, currently being reffered to as stealthjelly
Parts:
- J1: footprint Connector_PinSocket_2.54mm:PinSocket_1x04_P2.54mm_Vertical -> Connector_JST:JST_XH_B4B-XH-A_1x04_P2.50mm_Vertical
- turned J1 to 0 degrees
Other:
- board text added: "GND"
- board text added: "STRAIN"
- board text added: "VDDA"
