File: hardware/board files/strain gauges/BETA/minimal/minimal.kicad_sch (KiCad schematic)
At the start: 10 parts, among them J1 PR&J

Commit message: first revision of on board firmware, separate hardware and software folders
Parts:
- H1, H2, H3, H4: footprint MountingHole:MountingHole_2.7mm_Pad_Via -> MountingHole:MountingHole_3.2mm_M3_Pad_Via
Changed lines of the file:
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@@
     (pin "1")
     (instances
-      (project "strain gauge"
+      (project "minimal"
         (path "/4d674406-2df3-43ef-8583-5662efadc380"
           (reference "#PWR02") (unit 1)
@@
     (pin "2")
     (instances
-      (project "strain gauge"
+      (project "minimal"
         (path "/4d674406-2df3-43ef-8583-5662efadc380"
           (reference "R1") (unit 1)
@@
     (pin "5")
     (instances
-      (project "strain gauge"
+      (project "minimal"
         (path "/4d674406-2df3-43ef-8583-5662efadc380"
           (reference "U1") (unit 1)
@@
     (pin "2")
     (instances
-      (project "strain gauge"
+      (project "minimal"
         (path "/4d674406-2df3-43ef-8583-5662efadc380"
           (reference "R2") (unit 1)
@@
     (pin "4")
     (instances
-      (project "strain gauge"
+      (project "minimal"
         (path "/4d674406-2df3-43ef-8583-5662efadc380"
           (reference "J1") (unit 1)
@@
     (pin "2")
     (instances
-      (project "strain gauge"
+      (project "minimal"
         (path "/4d674406-2df3-43ef-8583-5662efadc380"
           (reference "R4") (unit 1)
@@
     (pin "1")
     (instances
-      (project "strain gauge"
+      (project "minimal"
         (path "/4d674406-2df3-43ef-8583-5662efadc380"
           (reference "#PWR01") (unit 1)
@@
       (effects (font (size 1.27 1.27)) (justify left))
     )
-    (property "Footprint" "MountingHole:MountingHole_2.7mm_Pad_Via" (at 134.62 38.735 0)
+    (property "Footprint" "MountingHole:MountingHole_3.2mm_M3_Pad_Via" (at 134.62 38.735 0)
       (effects (font (size 1.27 1.27)) hide)
     )
@@
     (pin "1")
     (instances
-      (project "strain gauge"
+      (project "minimal"
         (path "/4d674406-2df3-43ef-8583-5662efadc380"
           (reference "H3") (unit 1)
@@
     (pin "2")
     (instances
-      (project "strain gauge"
+      (project "minimal"
         (path "/4d674406-2df3-43ef-8583-5662efadc380"
           (reference "R3") (unit 1)
@@
     (pin "1")
     (instances
-      (project "strain gauge"
+      (project "minimal"
         (path "/4d674406-2df3-43ef-8583-5662efadc380"
           (reference "#PWR05") (unit 1)
@@
     (pin "1")
     (instances
-      (project "strain gauge"
+      (project "minimal"
         (path "/4d674406-2df3-43ef-8583-5662efadc380"
           (reference "#PWR06") (unit 1)
@@
       (effects (font (size 1.27 1.27)) (justify left))
     )
-    (property "Footprint" "MountingHole:MountingHole_2.7mm_Pad_Via" (at 134.62 33.655 0)
+    (property "Footprint" "MountingHole:MountingHole_3.2mm_M3_Pad_Via" (at 134.62 33.655 0)
       (effects (font (size 1.27 1.27)) hide)
     )
@@
     (pin "1")
     (instances
-      (project "strain gauge"
+      (project "minimal"
         (path "/4d674406-2df3-43ef-8583-5662efadc380"
           (reference "H2") (unit 1)
@@
       (effects (font (size 1.27 1.27)) (justify left))
     )
-    (property "Footprint" "MountingHole:MountingHole_2.7mm_Pad_Via" (at 134.62 28.575 0)
+    (property "Footprint" "MountingHole:MountingHole_3.2mm_M3_Pad_Via" (at 134.62 28.575 0)
       (effects (font (size 1.27 1.27)) hide)
     )
@@
     (pin "1")
     (instances
-      (project "strain gauge"
+      (project "minimal"
         (path "/4d674406-2df3-43ef-8583-5662efadc380"
           (reference "H1") (unit 1)
@@
     (pin "1")
     (instances
-      (project "strain gauge"
+      (project "minimal"
         (path "/4d674406-2df3-43ef-8583-5662efadc380"
           (reference "#PWR04") (unit 1)
@@
     (pin "1")
     (instances
-      (project "strain gauge"
+      (project "minimal"
         (path "/4d674406-2df3-43ef-8583-5662efadc380"
           (reference "#PWR03") (unit 1)
@@
       (effects (font (size 1.27 1.27)) (justify left))
     )
-    (property "Footprint" "MountingHole:MountingHole_2.7mm_Pad_Via" (at 134.62 43.815 0)
+    (property "Footprint" "MountingHole:MountingHole_3.2mm_M3_Pad_Via" (at 134.62 43.815 0)
       (effects (font (size 1.27 1.27)) hide)
     )
@@
     (pin "1")
     (instances
-      (project "strain gauge"
+      (project "minimal"
         (path "/4d674406-2df3-43ef-8583-5662efadc380"
           (reference "H4") (unit 1)

Commit message: added cad and stl files for initial test version of a modified stealthburner, currently being reffered to as stealthjelly
Parts:
- J1: footprint Connector_PinSocket_2.54mm:PinSocket_1x04_P2.54mm_Vertical -> Connector_JST:JST_XH_B4B-XH-A_1x04_P2.50mm_Vertical
Changed lines of the file:
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@@
       (effects (font (size 1.27 1.27)))
     )
-    (property "Footprint" "Connector_PinSocket_2.54mm:PinSocket_1x04_P2.54mm_Vertical" (at 44.45 32.385 0)
+    (property "Footprint" "Connector_JST:JST_XH_B4B-XH-A_1x04_P2.50mm_Vertical" (at 44.45 32.385 0)
       (effects (font (size 1.27 1.27)) hide)
     )
